Commit message: The model of robot is combined with gripper through constrain because it works better (for inverse kinematics calculations). The environment for gym is set up (needed to be checked).

File: models/ur10/ur10.urdf (robot description, URDF)
Before this commit: robot ur10, 9 links, 8 joints
Links:
- link base_link: geometry collision mesh filename=collision/Base.dae; visual mesh filename=visual/Base.dae
- link forearm_link: geometry collision mesh filename=collision/Forearm.dae; visual mesh filename=visual/Forearm.dae
- link shoulder_link: geometry collision mesh filename=collision/Shoulder.dae; visual mesh filename=visual/Shoulder.dae
- link upper_arm_link: geometry collision mesh filename=collision/UpperArm.dae; visual mesh filename=visual/UpperArm.dae
- link wrist_1_link: geometry collision mesh filename=collision/Wrist1.dae; visual mesh filename=visual/Wrist1.dae
- link wrist_2_link: geometry collision mesh filename=collision/Wrist2.dae; visual mesh filename=visual/Wrist2.dae
- link wrist_3_link: geometry collision mesh filename=collision/Wrist3.dae; visual mesh filename=visual/Wrist3.dae
Joints:
- joint world_joint: origin xyz=0.0 0.0 1.0 rpy=0.0 0.0 0.0 -> xyz=0.0 0.0 0.0 rpy=0.0 0.0 0.0

File: models/ur10_gripper/ur10_gripper.urdf (robot description, URDF)
Before this commit: robot ur10_robotiq_2f85, 17 links, 16 joints
Joints:
- joint finger_joint: type revolute -> fixed
- joint left_inner_finger_joint: type revolute -> fixed
- joint left_inner_knuckle_joint: type revolute -> fixed
- joint right_inner_finger_joint: type revolute -> fixed
- joint right_inner_knuckle_joint: type revolute -> fixed
- joint right_outer_knuckle_joint: type revolute -> fixed
