Commit message: The reward works not right, seems to require different function to compute. Size of the table is changed. TODO: check the penalties for the action.

File: models/table_custom/table.urdf (robot description, URDF)
Before this commit: robot table.urdf, 1 links, 0 joints
Links:
- link baseLink: geometry collision box size=3.0 3.0 0.05; visual mesh filename=table_custom/table.obj scale=0.1 0.1 0.58
